Commit message: Update with the latest f1tenth_gym

File: sim_ws/src/f1tenth_gym_ros/urdf/opp_racecar.xacro (robot description, xacro)
@@ -11,5 +11,6 @@
   <xacro:property name="laser_height" value="0.05" />
   <xacro:property name="laser_radius" value="0.026" />
-  <xacro:property name="car_name" value="opp_racecar" />
+  <xacro:arg name="car_name" default="opp_racecar" />
+  <xacro:property name="car_name" value="$(arg car_name)" />
   <material name="black">
     <color rgba="0.2 0.2 0.2 1."/>
